Commit message: motion planning

File: install/moveit_config/share/moveit_config/config/ur.ros2_control.xacro (robot description, xacro)
@@ -6,5 +6,5 @@
             <hardware>
                 <!-- By default, set up controllers for simulation. This won't work on real hardware -->
-                <plugin>mock_components/GenericSystem</plugin>
+                    <plugin>gz_ros2_control/GazeboSimSystem</plugin>
             </hardware>
             <joint name="shoulder_pan_joint">

File: install/moveit_config/share/moveit_config/config/ur.urdf.xacro (robot description, xacro)
@@ -2,8 +2,14 @@
 <robot xmlns:xacro="http://www.ros.org/wiki/xacro" name="ur">
     <xacro:arg name="initial_positions_file" default="initial_positions.yaml" />
+   <xacro:arg name="use_gazebo" default="true"/> <!-- Added missing argument -->
+   <xacro:arg name="robot_name" default="ur"/>
     <!-- Import ur urdf file -->
     <xacro:include filename="$(find ur_description)/urdf/ur.urdf.xacro" />
     <!-- Import control_xacro -->
-    <xacro:include filename="ur.ros2_control.xacro" />
-    <xacro:ur_ros2_control name="FakeSystem" initial_positions_file="$(arg initial_positions_file)"/>
+    <xacro:include filename="$(find moveit_config)/config/ur.ros2_control.xacro" />
+    <xacro:ur_ros2_control name="FakeSystem" initial_positions_file="$(find moveit_config)/config/initial_positions.yaml"/>
+    <xacro:include filename="$(find ur_description)/urdf/gazebo_sim_ros2_control.urdf.xacro" />
+   <xacro:load_gazebo_sim_ros2_control_plugin
+     robot_name="$(arg robot_name)"
+     use_gazebo="$(arg use_gazebo)"/>
 </robot>

File: install/robotiq_description/share/robotiq_description/urdf/robotiq_85_gripper.urdf.xacro (robot description, xacro)
@@ -102,4 +102,27 @@
                 </geometry>
             </collision>
+         <inertial>
+        <mass value="0.027309" />
+        <origin xyz="0.0 0.0 0.0" />
+        <inertia
+            ixx="0.0001"
+            ixy="0.0"
+            ixz="0.0"
+            iyy="0.0001"
+            iyz="0.0"
+            izz="0.0001" />
+    </inertial>
+        </link>
+        <link name="${prefix}robotiq_85_right_finger_link">
+            <visual>
+                <geometry>
+                    <mesh filename="package://robotiq_description/meshes/visual/robotiq_85_finger_link.dae"/>
+                </geometry>
+            </visual>
+            <collision>
+                <geometry>
+                    <mesh filename="package://robotiq_description/meshes/collision/robotiq_85_finger_link.stl"/>
+                </geometry>
+            </collision>
             <inertial>
                 <mass value="0.027309" />
@@ -110,23 +133,4 @@
             </inertial>
         </link>
-        <link name="${prefix}robotiq_85_right_finger_link">
-            <visual>
-                <geometry>
-                    <mesh filename="package://robotiq_description/meshes/visual/robotiq_85_finger_link.dae"/>
-                </geometry>
-            </visual>
-            <collision>
-                <geometry>
-                    <mesh filename="package://robotiq_description/meshes/collision/robotiq_85_finger_link.stl"/>
-                </geometry>
-            </collision>
-            <inertial>
-                <mass value="0.027309" />
-                <origin xyz="0.0 0.0 0.0" />
-                <inertia ixx = "0.000003" ixy = "-0.000002" ixz = "0.000000"
-                         iyx = "-0.000002" iyy = "0.000021" iyz = "0.000000"
-                         izx = "0.000000" izy = "0.000000" izz = "0.000020" />
-            </inertial>
-        </link>
         <joint name="${prefix}robotiq_85_left_inner_knuckle_joint" type="continuous">
             <parent link="${prefix}robotiq_85_base_link"/>
@@ -156,31 +160,39 @@
                 </geometry>
             </collision>
-            <inertial>
-                <mass value="0.029951" />
-                <origin xyz="0.0 0.0 0.0" />
-                <inertia ixx = "0.000039" ixy = "0.000000" ixz = "0.000000"
-                         iyx = "0.000000" iyy = "0.000005" iyz = "0.000000"
-                         izx = "0.000000" izy = "0.000000" izz = "0.000035" />
-            </inertial>
-        </link>
-        <link name="${prefix}robotiq_85_right_inner_knuckle_link">
-            <visual>
-                <geometry>
-                    <mesh filename="package://robotiq_description/meshes/visual/robotiq_85_inner_knuckle_link.dae"/>
-                </geometry>
-            </visual>
-            <collision>
-                <geometry>
-                    <mesh filename="package://robotiq_description/meshes/collision/robotiq_85_inner_knuckle_link.stl"/>
-                </geometry>
-            </collision>
-            <inertial>
-                <mass value="0.029951" />
-                <origin xyz="0.0 0.0 0.0" />
-                <inertia ixx = "0.000039" ixy = "0.000000" ixz = "0.000000"
-                         iyx = "0.000000" iyy = "0.000005" iyz = "0.000000"
-                         izx = "0.000000" izy = "0.000000" izz = "0.000035" />
-            </inertial>
-        </link>
+     <inertial>
+        <mass value="0.029951" />
+        <origin xyz="0.0 0.0 0.0" />
+        <inertia
+            ixx="0.0001"
+            ixy="0.0"
+            ixz="0.0"
+            iyy="0.0001"
+            iyz="0.0"
+            izz="0.0001" />
+    </inertial>
+        </link>
+<link name="${prefix}robotiq_85_right_inner_knuckle_link">
+    <visual>
+        <geometry>
+            <mesh filename="package://robotiq_description/meshes/visual/robotiq_85_inner_knuckle_link.dae"/>
+        </geometry>
+    </visual>
+    <collision>
+        <geometry>
+            <mesh filename="package://robotiq_description/meshes/collision/robotiq_85_inner_knuckle_link.stl"/>
+        </geometry>
+    </collision>
+        <inertial>
+        <mass value="0.027309" />
+        <origin xyz="0.0 0.0 0.0" />
+        <inertia
+            ixx="0.0001"
+            ixy="0.0"
+            ixz="0.0"
+            iyy="0.0001"
+            iyz="0.0"
+            izz="0.0001" />
+    </inertial>
+</link>
         <joint name="${prefix}robotiq_85_left_finger_tip_joint" type="continuous">
             <parent link="${prefix}robotiq_85_left_inner_knuckle_link"/>
@@ -210,4 +222,27 @@
                 </geometry>
             </collision>
+        <inertial>
+        <mass value="0.027309" />
+        <origin xyz="0.0 0.0 0.0" />
+        <inertia
+            ixx="0.0001"
+            ixy="0.0"
+            ixz="0.0"
+            iyy="0.0001"
+            iyz="0.0"
+            izz="0.0001" />
+    </inertial>
+        </link>
+        <link name="${prefix}robotiq_85_right_finger_tip_link">
+            <visual>
+                <geometry>
+                    <mesh filename="package://robotiq_description/meshes/visual/robotiq_85_finger_tip_link.dae"/>
+                </geometry>
+            </visual>
+            <collision>
+                <geometry>
+                    <mesh filename="package://robotiq_description/meshes/collision/robotiq_85_finger_tip_link.stl"/>
+                </geometry>
+            </collision>
             <inertial>
                 <mass value="0.019555" />
@@ -218,23 +253,4 @@
             </inertial>
         </link>
-        <link name="${prefix}robotiq_85_right_finger_tip_link">
-            <visual>
-                <geometry>
-                    <mesh filename="package://robotiq_description/meshes/visual/robotiq_85_finger_tip_link.dae"/>
-                </geometry>
-            </visual>
-            <collision>
-                <geometry>
-                    <mesh filename="package://robotiq_description/meshes/collision/robotiq_85_finger_tip_link.stl"/>
-                </geometry>
-            </collision>
-            <inertial>
-                <mass value="0.019555" />
-                <origin xyz="0.0 0.0 0.0" />
-                <inertia ixx = "0.000002" ixy = "0.000000" ixz = "0.000000"
-                         iyx = "0.000000" iyy = "0.000005" iyz = "0.000000"
-                         izx = "0.000000" izy = "0.000000" izz = "0.000006" />
-            </inertial>
-        </link>
         <xacro:robotiq_85_gripper_transmission prefix="${prefix}" />
     </xacro:macro>

File: install/ur_description/share/ur_description/urdf/ur.urdf.xacro (robot description, xacro)
@@ -35,4 +35,6 @@
      <origin xyz="0 0 0" rpy="0 0 0" /> <!-- Position robot in the world -->
    </xacro:ur_robot>
+    <xacro:include filename="$(find moveit_config)/config/ur.ros2_control.xacro" />
+    <xacro:ur_ros2_control name="FakeSystem" initial_positions_file="$(find moveit_config)/config/initial_positions.yaml"/>
    <!-- Include Gazebo Simulation Control Plugin -->
    <!-- <xacro:include filename="$(find ur_description)/urdf/gazebo_sim_ros2_control.urdf.xacro" />
